File: Wild Spy Open Source Timer.kicad_pcb (KiCad board)
At the start: 2 copper layers, 30 x 32.8 mm, 74 parts, among them Q1 AO3415, Q2 AO3415, Q3 AO3415, Q4 AO3415, Q5 AO3415, Q6 AO3415, SW1 SW_PUSH, SW2 ORD213, U1 DS3232SN, U2 TPS70933DBVR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

Commit message: Fixed battery volrage measurement issue in hardware.
Parts:
- added Q7: BSH103, OSTFootprints:SOT-23-HandSoldering, B.Cu at (195.1, 113.2)
- added R12: 100k, Resistors_SMD:R_0603_HandSoldering, B.Cu at (192.4, 120.9)
- added REF**: VIA-0.3mm, MC_Footprint:VIA-0.3mm, F.Cu at (214.1, 124.8)
- added REF**: VIA-0.3mm, MC_Footprint:VIA-0.3mm, F.Cu at (198.5, 124.0)
- added REF**: VIA-0.3mm, MC_Footprint:VIA-0.3mm, F.Cu at (201.7, 121.4)
- added REF**: VIA-0.3mm, MC_Footprint:VIA-0.3mm, F.Cu at (197.1, 117.0)
- added REF**: VIA-0.3mm, MC_Footprint:VIA-0.3mm, F.Cu at (192.1, 125.9)
- added REF**: VIA-0.3mm, MC_Footprint:VIA-0.3mm, F.Cu at (208.8, 119.3)
- added REF**: VIA-0.3mm, MC_Footprint:VIA-0.3mm, F.Cu at (214.2, 112.5)
- added REF**: VIA-0.3mm, MC_Footprint:VIA-0.3mm, F.Cu at (214.2, 113.8)
- added REF**: VIA-0.3mm, MC_Footprint:VIA-0.3mm, F.Cu at (211.0, 106.5)
- added REF**: VIA-0.3mm, MC_Footprint:VIA-0.3mm, F.Cu at (192.7, 107.3)
- added REF**: VIA-0.3mm, MC_Footprint:VIA-0.3mm, F.Cu at (193.2, 99.0)
- added REF**: VIA-0.3mm, MC_Footprint:VIA-0.3mm, F.Cu at (193.0, 97.1)
- moved REF** 7.43 mm to (207.5, 117.4)
- moved REF** 6.42 mm to (207.8, 121.2)
- moved REF** 5.76 mm to (198.1, 119.6)
- moved REF** 4.82 mm to (214.5, 116.0)
- moved REF** 4.36 mm to (218.2, 111.7)
- moved JP1 4.10 mm to (212.5, 118.8)
- moved Battery1 2.56 mm to (217.4, 125.5), turned to 180 degrees
- moved REF** 2.22 mm to (212.8, 124.2)
- moved REF** 2.18 mm to (195.6, 114.5)
- moved REF** 1.86 mm to (194.3, 110.8)
- moved R3 1.56 mm to (211.7, 116.7)
- moved R8 1.48 mm to (211.7, 118.3)
- moved REF** 1.18 mm to (196.3, 122.6)
- moved REF** 0.83 mm to (192.6, 124.7)
- moved REF** 0.75 mm to (198.0, 112.8)
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Connections:
- Q6 pad 1: /~BatMeasureEn -> Net-(Q6-Pad1)
- U5 pad 14: /~BatMeasureEn -> Net-(U5-Pad14)
- U5 pad 27: Net-(U5-Pad27) -> /BatMeasureEn
Routing:
- net Net-(Q6-Pad1): track 0.00 -> 39.4 mm, vias 0 -> 2
- net GND: track 29.4 -> 52.2 mm
- net VAA: track 13.4 -> 34.9 mm, vias 2 -> 3
- net /BatMeasureEn: track 0.00 -> 20.4 mm, vias 0 -> 2
- net /~BatMeasureEn: track 7.53 -> 0.00 mm
- net /BAT+: track 3.48 -> 8.84 mm
- net /SCL: track 22.8 -> 25.5 mm
- net /SDA: track 20.0 -> 22.0 mm
- net +5V: track 9.70 -> 11.4 mm
- net Net-(Q6-Pad3): track 7.25 -> 5.60 mm
- net Net-(U5-Pad14): track 0.00 -> 0.97 mm, vias 0 -> 1
- net VCC: track 72.8 -> 72.2 mm
- net /LED: track 8.67 -> 8.11 mm
Other:
- board text added: "Rev1.1"
- board text removed: "HBowman"
- board text removed: "MCochrane"
- board text removed: "Rev1"

Commit message: Manufacturing outputs for Rev1.1
Changed lines of the file:
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@@
     (links 164)
     (no_connects 2)
-    (area 188.924999 94.158999 219.075001 127.075001)
+    (area 20.235999 76.034899 238.785402 191.255001)
     (thickness 1.6)
     (drawings 501)
-    (tracks 541)
+    (tracks 540)
     (zones 0)
     (modules 88)
@@
   (layers
     (0 F.Cu signal)
-    (31 B.Cu signal hide)
+    (31 B.Cu signal)
     (32 B.Adhes user hide)
     (33 F.Adhes user hide)
@@
       (drillshape 0)
       (scaleselection 1)
-      (outputdirectory "Manufacturing Outputs/Rev1/"))
+      (outputdirectory "Manufacturing Outputs/Rev1.1/"))
   )
   (net 0 "")
@@
   (segment (start 200.330579 114.70161) (end 199.8345 115.197689) (width 0.2032) (layer F.Cu) (net 51))
   (segment (start 199.8345 115.197689) (end 199.8345 115.514703) (width 0.2032) (layer F.Cu) (net 51))
-  (segment (start 190.181 113.792) (end 190.119 113.73) (width 0.2032) (layer B.Cu) (net 51))
   (segment (start 193.929 114.427) (end 193.294 113.792) (width 0.2032) (layer F.Cu) (net 51))
   (via (at 191.389 113) (size 0.6) (drill 0.3) (layers F.Cu B.Cu) (net 51))
